File: kicad/pulse_generator/pulse_generator.kicad_sch (KiCad schematic)
At the start: 12 parts, among them J1 Power, J2 Digital/PWM, J3 Analog, J4 Digital/PWM, J5 input via pullup r, J6 pulse_output, Q1 BS170, U1 Digilent_Pmod_KYPD:_16-Button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

Commit message: UPDATE
Parts:
- removed DS1: MC42005A6W-BNMLW-V2, MC42005A6WBNMLWV2, symbol SamacSys_Parts:MC42005A6W-BNMLW-V2
- added DS1: FC2004B01-FHYYBW-51SE, Connector_PinHeader_2.54mm:PinHeader_1x16_P2.54mm_Vertical, symbol Display_Graphic:FC2004B01-FHYYBW-51SE
- added RV1: R_Potentiometer, symbol Device:R_Potentiometer
Connections:
- net A0: now also DS1.4 (RS)
- net A1: now also DS1.6 (E)
- net A2: now also DS1.7 (DB0)
- net A3: now also DS1.8 (DB1)
- net GND: now also DS1.5 (R/W)
- net SCL/A5: now also DS1.10 (DB3)
- net SDA/A4: now also DS1.9 (DB2)
- new net: DS1.2 (VDD), RV1.1
- new net: DS1.3 (V0), RV1.2
- new net: DS1.1 (VSS), RV1.3
Other:
- moved on the sheet: D1, J1, J2, J3, J4, J5, J6, Q1, R1, R2

Commit message: u
Connections:
- net *10: now also U1.4 (COL1)
- net *11: now also U1.3 (COL2)
- net *5: now also U1.10 (ROW1)
- net *6: now also U1.9 (ROW2)
- net +5V: now also DS1.15 (LED+), DS1.2 (VDD), RV1.1, U1.12 (VCC), U1.6 (VCC)
- net 12: now also U1.2 (COL3)
- net 13: now also U1.1 (COL4)
- net 7: now also U1.8 (ROW3)
- net 8: now also U1.7 (ROW4)
- net A2: now also DS1.14 (DB7); no longer DS1.7 (DB0)
- net A3: now also DS1.13 (DB6); no longer DS1.8 (DB1)
- net GND: now also DS1.1 (VSS), DS1.10 (DB3), DS1.16 (LED-), DS1.7 (DB0), DS1.8 (DB1), DS1.9 (DB2), RV1.3, U1.11 (GND), U1.5 (GND)
- net SCL/A5: now also DS1.11 (DB4); no longer DS1.10 (DB3)
- net SDA/A4: now also DS1.12 (DB5); no longer DS1.9 (DB2)
Other:
- note added: "ARDUINO UNO REV3"
- moved on the sheet: RV1, U1

Commit message: u
Connections:
- net *9: no longer J2.9 (Pin_9), J4.4 (Pin_4)
Changed lines of the file:
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@@
     (stroke (width 0) (type default))
-  )
-  (wire (pts (xy 129.54 50.8) (xy 148.59 50.8))
-    (stroke (width 0) (type solid))
   )
   (wire (pts (xy 185.42 66.04) (xy 185.42 60.96))
@@
   (wire (pts (xy 132.08 38.1) (xy 132.08 55.88))
     (stroke (width 0) (type solid))
-  )
-  (wire (pts (xy 148.59 50.8) (xy 148.59 71.12))
-    (stroke (width 0) (type default))
   )
   (wire (pts (xy 81.28 68.58) (xy 101.6 68.58))
@@
     (stroke (width 0) (type solid))
   )
-  (wire (pts (xy 129.54 71.12) (xy 148.59 71.12))
-    (stroke (width 0) (type default))
-  )
   (wire (pts (xy 165.1 54.61) (xy 172.72 54.61))

Commit message: u
Parts:
- removed D1: L-53GD, symbol Device:LED
- removed R1: 140, symbol Device:R
Connections:
- net *3 is gone; now on net GND: J4.5 (Pin_5)
- net GND: now also J2.9 (Pin_9), J4.4 (Pin_4)
- no-connect marks 1 -> 3
Other:
- note removed: "Possible RC in parallel over diode"
Changed lines of the file:
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@@
   (junction (at 99.06 50.8) (diameter 1.016) (color 0 0 0 0)
   )
+  (junction (at 160.02 73.66) (diameter 0) (color 0 0 0 0)
+  )
+  (junction (at 132.08 50.8) (diameter 0) (color 0 0 0 0)
+  )
   (junction (at 147.32 111.76) (diameter 0) (color 0 0 0 0)
   )
@@
   (junction (at 62.23 38.1) (diameter 0) (color 0 0 0 0)
   )
+  (no_connect (at 142.24 81.28))
+  (no_connect (at 142.24 78.74))
   (no_connect (at 101.6 35.56))
   (wire (pts (xy 129.54 81.28) (xy 142.24 81.28))
@@
     (stroke (width 0) (type default))
   )
+  (wire (pts (xy 129.54 73.66) (xy 160.02 73.66))
+    (stroke (width 0) (type default))
+  )
   (wire (pts (xy 78.74 73.66) (xy 101.6 73.66))
     (stroke (width 0) (type default))
@@
     (stroke (width 0) (type default))
   )
-  (wire (pts (xy 185.42 81.28) (xy 185.42 83.82))
-    (stroke (width 0) (type default))
-  )
   (wire (pts (xy 129.54 30.48) (xy 142.24 30.48))
     (stroke (width 0) (type solid))
@@
     (stroke (width 0) (type default))
   )
+  (wire (pts (xy 129.54 50.8) (xy 132.08 50.8))
+    (stroke (width 0) (type default))
+  )
   (wire (pts (xy 74.93 68.58) (xy 74.93 66.04))
     (stroke (width 0) (type default))
@@
     (stroke (width 0) (type solid))
   )
+  (wire (pts (xy 129.54 71.12) (xy 160.02 71.12))
+    (stroke (width 0) (type default))
+  )
   (wire (pts (xy 96.52 30.48) (xy 96.52 45.72))
     (stroke (width 0) (type solid))
@@
     (stroke (width 0) (type default))
   )
+  (wire (pts (xy 132.08 50.8) (xy 132.08 55.88))
+    (stroke (width 0) (type solid))
+  )
   (wire (pts (xy 129.54 40.64) (xy 157.48 40.64))
     (stroke (width 0) (type solid))
@@
     (stroke (width 0) (type default))
   )
-  (wire (pts (xy 185.42 91.44) (xy 185.42 93.98))
-    (stroke (width 0) (type default))
-  )
   (wire (pts (xy 129.54 66.04) (xy 165.1 66.04))
     (stroke (width 0) (type solid))
@@
     (stroke (width 0) (type default))
   )
-  (wire (pts (xy 129.54 73.66) (xy 185.42 73.66))
-    (stroke (width 0) (type default))
-  )
   (wire (pts (xy 185.42 24.13) (xy 185.42 33.02))
     (stroke (width 0) (type default))
   )
-  (wire (pts (xy 132.08 38.1) (xy 132.08 55.88))
+  (wire (pts (xy 132.08 38.1) (xy 132.08 50.8))
     (stroke (width 0) (type solid))
   )
@@
     (stroke (width 0) (type default))
   )
+  (wire (pts (xy 160.02 71.12) (xy 160.02 73.66))
+    (stroke (width 0) (type default))
+  )
   (wire (pts (xy 86.36 40.64) (xy 101.6 40.64))
     (stroke (width 0) (type solid))
@@
   )
   (text "ARDUINO UNO REV3\n" (at 116.84 64.77 90)
-    (effects (font (size 1.27 1.27)) (justify left bottom))
-  )
-  (text "Possible RC in parallel\nover diode" (at 189.23 87.63 0)
     (effects (font (size 1.27 1.27)) (justify left bottom))
   )
@@
     )
   )
+  (symbol (lib_name "GND_2") (lib_id "power:GND") (at 160.02 73.66 0) (unit 1)
+    (in_bom yes) (on_board yes) (dnp no) (fields_autoplaced)
+    (property "Reference" "#PWR06" (at 160.02 80.01 0)
+      (effects (font (size 1.27 1.27)) hide)
+    )
+    (property "Value" "GND" (at 160.02 78.74 0)
+      (effects (font (size 1.27 1.27)))
+    )
+    (property "Footprint" "" (at 160.02 73.66 0)
+      (effects (font (size 1.27 1.27)) hide)
+    )
+    (property "Datasheet" "" (at 160.02 73.66 0)
+      (effects (font (size 1.27 1.27)) hide)
+    )
+    (pin "1")
+    (instances
+      (project "pulse_generator"
+        (path "/e63e39d7-6ac0-4ffd-8aa3-1841a4541b55"
+          (reference "#PWR06") (unit 1)
+        )
+      )
+    )
+  )
   (symbol (lib_id "power:VCC") (at 93.98 30.48 0) (unit 1)
     (in_bom yes) (on_board yes) (dnp no)
@@
         (path "/e63e39d7-6ac0-4ffd-8aa3-1841a4541b55"
           (reference "#PWR01") (unit 1)
-        )
-      )
-    )
-  )
-  (symbol (lib_id "Device:R") (at 185.42 77.47 0) (unit 1)
-    (in_bom yes) (on_board yes) (dnp no) (fields_autoplaced)
-    (property "Reference" "R1" (at 187.96 76.835 0)
-      (effects (font (size 1.27 1.27)) (justify left))
-    )
-    (property "Value" "140" (at 187.96 79.375 0)
-      (effects (font (size 1.27 1.27)) (justify left))
-    )
-    (property "Footprint" "" (at 183.642 77.47 90)
-      (effects (font (size 1.27 1.27)) hide)
-    )
-    (property "Datasheet" "~" (at 185.42 77.47 0)
-      (effects (font (size 1.27 1.27)) hide)
-    )
-    (pin "1")
-    (pin "2")
-    (instances
-      (project "pulse_generator"
-        (path "/e63e39d7-6ac0-4ffd-8aa3-1841a4541b55"
-          (reference "R1") (unit 1)
-        )
-      )
-    )
-  )
-  (symbol (lib_id "Device:LED") (at 185.42 87.63 90) (unit 1)
-    (in_bom yes) (on_board yes) (dnp no) (fields_autoplaced)
-    (property "Reference" "D1" (at 189.23 88.5825 90)
-      (effects (font (size 1.27 1.27)) (justify right))
-    )
-    (property "Value" "L-53GD" (at 189.23 91.1225 90)
-      (effects (font (size 1.27 1.27)) (justify right))
-    )
-    (property "Footprint" "" (at 185.42 87.63 0)
-      (effects (font (size 1.27 1.27)) hide)
-    )
-    (property "Datasheet" "https://docs.rs-online.com/4066/0900766b8151e408.pdf" (at 185.42 87.63 0)
-      (effects (font (size 1.27 1.27)) hide)
-    )
-    (pin "1")
-    (pin "2")
-    (instances
-      (project "pulse_generator"
-        (path "/e63e39d7-6ac0-4ffd-8aa3-1841a4541b55"
-          (reference "D1") (unit 1)
         )
       )
@@
         )
       )
-    )
-  )
-  (symbol (lib_name "GND_1") (lib_id "power:GND") (at 185.42 93.98 0) (unit 1)
-    (in_bom yes) (on_board yes) (dnp no) (fields_autoplaced)
-    (property "Reference" "#PWR06" (at 185.42 100.33 0)
-      (effects (font (size 1.27 1.27)) hide)
-    )
-    (property "Value" "GND" (at 185.42 99.06 0)
-      (effects (font (size 1.27 1.27)))
-    )
-    (property "Footprint" "" (at 185.42 93.98 0)
-      (effects (font (size 1.27 1.27)) hide)
-    )
-    (property "Datasheet" "" (at 185.42 93.98 0)
-      (effects (font (size 1.27 1.27)) hide)
-    )
-    (pin "1")
-    (instances
-      (project "pulse_generator"
-        (path "/e63e39d7-6ac0-4ffd-8aa3-1841a4541b55"
-          (reference "#PWR06") (unit 1)
-        )
-      )
